Commit message: fixed colors

File: robot_description/urdf/materials.xacro (robot description, xacro)
@@ -4,12 +4,12 @@
   <color rgba="0.700 0.700 0.700 1.000"/>
 </material>
-<material name="opaque515151">
-  <color rgba="0.2 0.2 0.2 1.0"/>
+<material name="red">
+  <color rgba="1.0 0.0 0.0 1.0"/>
 </material>
-<material name="opaque202209238">
-  <color rgba="0.792156862745098 0.8196078431372549 0.9333333333333333 1.0"/>
+<material name="black">
+  <color rgba="0.0 0.0 0.0 1.0"/>
 </material>
-<material name="abs_white">
-  <color rgba="0.9647058823529412 0.9647058823529412 0.9529411764705882 1.0"/>
+<material name="blue">
+  <color rgba="0.0 0.0 1.0 1.0"/>
 </material>
 </robot>

File: robot_description/urdf/robot.xacro (robot description, xacro)
@@ -15,5 +15,5 @@
       <mesh filename="package://robot_description/meshes/base_link.stl" scale="0.001 0.001 0.001"/>
     </geometry>
-    <material name="opaque515151"/>
+    <material name="red"/>
   </visual>
   <collision>
@@ -35,5 +35,5 @@
       <mesh filename="package://robot_description/meshes/wheel_back_left_1.stl" scale="0.001 0.001 0.001"/>
     </geometry>
-    <material name="opaque202209238"/>
+    <material name="black"/>
   </visual>
   <collision>
@@ -55,5 +55,5 @@
       <mesh filename="package://robot_description/meshes/wheel_back_right_1.stl" scale="0.001 0.001 0.001"/>
     </geometry>
-    <material name="opaque202209238"/>
+    <material name="black"/>
   </visual>
   <collision>
@@ -75,5 +75,5 @@
       <mesh filename="package://robot_description/meshes/wheel_front_right_1.stl" scale="0.001 0.001 0.001"/>
     </geometry>
-    <material name="opaque202209238"/>
+    <material name="black"/>
   </visual>
   <collision>
@@ -95,5 +95,5 @@
       <mesh filename="package://robot_description/meshes/wheel_front_left_1.stl" scale="0.001 0.001 0.001"/>
     </geometry>
-    <material name="opaque202209238"/>
+    <material name="black"/>
   </visual>
   <collision>
@@ -115,5 +115,5 @@
       <mesh filename="package://robot_description/meshes/lidar_1.stl" scale="0.001 0.001 0.001"/>
     </geometry>
-    <material name="abs_white"/>
+    <material name="blue"/>
   </visual>
   <collision>
