Commit message: teleop functional

File: robot_description/urdf/robot.xacro (robot description, xacro)
@@ -4,8 +4,15 @@
 <xacro:include filename="$(find robot_description)/urdf/robot.trans" />
 <xacro:include filename="$(find robot_description)/urdf/robot.gazebo" />
+<link name="robot_footprint"></link>
+  <joint name="robot_footprint_joint" type="fixed">
+    <origin xyz="0 0 0" rpy="0 0 0" />
+    <parent link="robot_footprint" />
+    <child link="base_link" />
+  </joint>
 <link name="base_link">
   <inertial>
     <origin xyz="-0.2022009373759702 -0.004939439834032545 0.41355366312881875" rpy="0 0 0"/>
-    <mass value="224.78888813493901"/>
+    <!-- <mass value="224.78888813493901"/> -->
+    <mass value="100.78888813493901"/>
     <inertia ixx="10.277979" iyy="24.4356" izz="25.482363" ixy="0.003732" iyz="-0.001902" ixz="3.810092"/>
   </inertial>
@@ -107,5 +114,5 @@
   <inertial>
     <origin xyz="2.534804336429275e-07 -3.095004238833077e-07 0.02952388194216904" rpy="0 0 0"/>
-    <mass value="2.3275293008071234"/>
+    <mass value="60.3275293008071234"/>
     <inertia ixx="0.001597" iyy="0.001597" izz="0.001837" ixy="-0.0" iyz="0.0" ixz="0.0"/>
   </inertial>
@@ -134,5 +141,5 @@
   <parent link="base_link"/>
   <child link="wheel_back_right_1"/>
-  <axis xyz="0.0 1.0 0.0"/>
+  <axis xyz="0.0 -1.0 0.0"/>
 </joint>
 <joint name="joint_front_right" type="continuous">
@@ -140,5 +147,5 @@
   <parent link="base_link"/>
   <child link="wheel_front_right_1"/>
-  <axis xyz="0.0 1.0 0.0"/>
+  <axis xyz="0.0 -1.0 0.0"/>
 </joint>
 <joint name="joint_front_left" type="continuous">

Commit message: hokuyo laser added

File: robot_description/urdf/robot.xacro (robot description, xacro)
@@ -14,5 +14,5 @@
     <origin xyz="-0.2022009373759702 -0.004939439834032545 0.41355366312881875" rpy="0 0 0"/>
     <!-- <mass value="224.78888813493901"/> -->
-    <mass value="100.78888813493901"/>
+    <mass value="150.78888813493901"/>
     <inertia ixx="10.277979" iyy="24.4356" izz="25.482363" ixy="0.003732" iyz="-0.001902" ixz="3.810092"/>
   </inertial>
@@ -114,5 +114,5 @@
   <inertial>
     <origin xyz="2.534804336429275e-07 -3.095004238833077e-07 0.02952388194216904" rpy="0 0 0"/>
-    <mass value="60.3275293008071234"/>
+    <mass value="100.3275293008071234"/>
     <inertia ixx="0.001597" iyy="0.001597" izz="0.001837" ixy="-0.0" iyz="0.0" ixz="0.0"/>
   </inertial>

Commit message: wheel direction fixed

File: robot_description/urdf/robot.xacro (robot description, xacro)
@@ -2,5 +2,5 @@
 <robot name="robot" xmlns:xacro="http://www.ros.org/wiki/xacro">
 <xacro:include filename="$(find robot_description)/urdf/materials.xacro" />
-<xacro:include filename="$(find robot_description)/urdf/robot.trans" />
+<!-- <xacro:include filename="$(find robot_description)/urdf/robot.trans" /> -->
 <xacro:include filename="$(find robot_description)/urdf/robot.gazebo" />
 <link name="robot_footprint"></link>
@@ -135,5 +135,7 @@
   <parent link="base_link"/>
   <child link="wheel_back_left_1"/>
-  <axis xyz="-0.0 -1.0 -0.0"/>
+  <axis xyz="0.0 1.0 0.0"/>
+  <limit effort="10000" velocity="1000"/>
+  <joint_properties damping="1.0" friction="1.0"/>
 </joint>
 <joint name="joint_back_right" type="continuous">
@@ -141,5 +143,7 @@
   <parent link="base_link"/>
   <child link="wheel_back_right_1"/>
-  <axis xyz="0.0 -1.0 0.0"/>
+  <axis xyz="0.0 1.0 0.0"/>
+  <limit effort="10000" velocity="1000"/>
+  <joint_properties damping="1.0" friction="1.0"/>
 </joint>
 <joint name="joint_front_right" type="continuous">
@@ -147,5 +151,7 @@
   <parent link="base_link"/>
   <child link="wheel_front_right_1"/>
-  <axis xyz="0.0 -1.0 0.0"/>
+  <axis xyz="0.0 1.0 0.0"/>
+  <limit effort="10000" velocity="1000"/>
+  <joint_properties damping="1.0" friction="1.0"/>
 </joint>
 <joint name="joint_front_left" type="continuous">
@@ -153,5 +159,7 @@
   <parent link="base_link"/>
   <child link="wheel_front_left_1"/>
-  <axis xyz="-0.0 -1.0 -0.0"/>
+  <axis xyz="0.0 1.0 0.0"/>
+  <limit effort="10000" velocity="1000"/>
+  <joint_properties damping="1.0" friction="1.0"/>
 </joint>
 <joint name="joint_lidar" type="fixed">

Commit message: robot moves to target but jumpy, inaccurate

File: robot_description/urdf/robot.xacro (robot description, xacro)
@@ -13,6 +13,6 @@
   <inertial>
     <origin xyz="-0.2022009373759702 -0.004939439834032545 0.41355366312881875" rpy="0 0 0"/>
-    <!-- <mass value="224.78888813493901"/> -->
-    <mass value="150.78888813493901"/>
+    <mass value="224.78888813493901"/>
+    <!-- <mass value="150.78888813493901"/> -->
     <inertia ixx="10.277979" iyy="24.4356" izz="25.482363" ixy="0.003732" iyz="-0.001902" ixz="3.810092"/>
   </inertial>

Commit message: follow waypoints functional

File: robot_description/urdf/robot.xacro (robot description, xacro)
@@ -12,8 +12,8 @@
 <link name="base_link">
   <inertial>
-    <origin xyz="-0.2022009373759702 -0.004939439834032545 0.41355366312881875" rpy="0 0 0"/>
-    <mass value="224.78888813493901"/>
-    <!-- <mass value="150.78888813493901"/> -->
-    <inertia ixx="10.277979" iyy="24.4356" izz="25.482363" ixy="0.003732" iyz="-0.001902" ixz="3.810092"/>
+    <origin xyz="0.20220093737597014 0.004939439834032356 0.41355366312881875" rpy="0 0 0"/>
+    <mass value="150.78888813493904"/>
+    <!-- <mass value="224.78888813493904"/> -->
+    <inertia ixx="10.277979" iyy="24.4356" izz="25.482363" ixy="0.003732" iyz="0.001902" ixz="-3.810092"/>
   </inertial>
   <visual>
@@ -33,10 +33,10 @@
 <link name="wheel_back_left_1">
   <inertial>
-    <origin xyz="1.7376132144253376e-08 -0.002997907926125032 -2.495734152674345e-07" rpy="0 0 0"/>
+    <origin xyz="-1.7376132255275678e-08 0.002997907926125032 -2.4957341521192333e-07" rpy="0 0 0"/>
     <mass value="18.850995744913625"/>
-    <inertia ixx="0.224929" iyy="0.359773" izz="0.224929" ixy="0.0" iyz="-0.0" ixz="0.0"/>
+    <inertia ixx="0.224929" iyy="0.359773" izz="0.224929" ixy="0.0" iyz="0.0" ixz="-0.0"/>
   </inertial>
   <visual>
-    <origin xyz="-0.353612 0.345039 -0.173506" rpy="0 0 0"/>
+    <origin xyz="0.353612 -0.345039 -0.173506" rpy="0 0 0"/>
     <geometry>
       <mesh filename="package://robot_description/meshes/wheel_back_left_1.stl" scale="0.001 0.001 0.001"/>
@@ -45,5 +45,5 @@
   </visual>
   <collision>
-    <origin xyz="-0.353612 0.345039 -0.173506" rpy="0 0 0"/>
+    <origin xyz="0.353612 -0.345039 -0.173506" rpy="0 0 0"/>
     <geometry>
       <mesh filename="package://robot_description/meshes/wheel_back_left_1.stl" scale="0.001 0.001 0.001"/>
@@ -53,10 +53,10 @@
 <link name="wheel_back_right_1">
   <inertial>
-    <origin xyz="1.737613286589834e-08 0.0025020920738725305 -2.495734181817699e-07" rpy="0 0 0"/>
+    <origin xyz="-1.737613281038719e-08 -0.0025020920738726415 -2.4957341812625877e-07" rpy="0 0 0"/>
     <mass value="18.85099574491358"/>
-    <inertia ixx="0.224929" iyy="0.359773" izz="0.224929" ixy="0.0" iyz="-0.0" ixz="0.0"/>
+    <inertia ixx="0.224929" iyy="0.359773" izz="0.224929" ixy="0.0" iyz="0.0" ixz="-0.0"/>
   </inertial>
   <visual>
-    <origin xyz="-0.353612 -0.334961 -0.173506" rpy="0 0 0"/>
+    <origin xyz="0.353612 0.334961 -0.173506" rpy="0 0 0"/>
     <geometry>
       <mesh filename="package://robot_description/meshes/wheel_back_right_1.stl" scale="0.001 0.001 0.001"/>
@@ -65,5 +65,5 @@
   </visual>
   <collision>
-    <origin xyz="-0.353612 -0.334961 -0.173506" rpy="0 0 0"/>
+    <origin xyz="0.353612 0.334961 -0.173506" rpy="0 0 0"/>
     <geometry>
       <mesh filename="package://robot_description/meshes/wheel_back_right_1.stl" scale="0.001 0.001 0.001"/>
@@ -73,10 +73,10 @@
 <link name="wheel_front_right_1">
   <inertial>
-    <origin xyz="-4.0520683738942687e-07 0.0025020920738714203 -2.495734135465888e-07" rpy="0 0 0"/>
+    <origin xyz="4.0520683730616014e-07 -0.0025020920738715313 -2.495734135188332e-07" rpy="0 0 0"/>
     <mass value="18.850995744914012"/>
-    <inertia ixx="0.224929" iyy="0.359773" izz="0.224929" ixy="0.0" iyz="-0.0" ixz="0.0"/>
+    <inertia ixx="0.224929" iyy="0.359773" izz="0.224929" ixy="0.0" iyz="0.0" ixz="-0.0"/>
   </inertial>
   <visual>
-    <origin xyz="0.223665 -0.334961 -0.173506" rpy="0 0 0"/>
+    <origin xyz="-0.223665 0.334961 -0.173506" rpy="0 0 0"/>
     <geometry>
       <mesh filename="package://robot_description/meshes/wheel_front_right_1.stl" scale="0.001 0.001 0.001"/>
@@ -85,5 +85,5 @@
   </visual>
   <collision>
-    <origin xyz="0.223665 -0.334961 -0.173506" rpy="0 0 0"/>
+    <origin xyz="-0.223665 0.334961 -0.173506" rpy="0 0 0"/>
     <geometry>
       <mesh filename="package://robot_description/meshes/wheel_front_right_1.stl" scale="0.001 0.001 0.001"/>
@@ -93,10 +93,10 @@
 <link name="wheel_front_left_1">
   <inertial>
-    <origin xyz="-4.052068346416249e-07 -0.0029979079261240327 -2.4957341610010175e-07" rpy="0 0 0"/>
+    <origin xyz="4.0520683466938046e-07 0.0029979079261240327 -2.495734160723462e-07" rpy="0 0 0"/>
     <mass value="18.850995744914055"/>
-    <inertia ixx="0.224929" iyy="0.359773" izz="0.224929" ixy="0.0" iyz="-0.0" ixz="0.0"/>
+    <inertia ixx="0.224929" iyy="0.359773" izz="0.224929" ixy="0.0" iyz="0.0" ixz="-0.0"/>
   </inertial>
   <visual>
-    <origin xyz="0.223665 0.345039 -0.173506" rpy="0 0 0"/>
+    <origin xyz="-0.223665 -0.345039 -0.173506" rpy="0 0 0"/>
     <geometry>
       <mesh filename="package://robot_description/meshes/wheel_front_left_1.stl" scale="0.001 0.001 0.001"/>
@@ -105,5 +105,5 @@
   </visual>
   <collision>
-    <origin xyz="0.223665 0.345039 -0.173506" rpy="0 0 0"/>
+    <origin xyz="-0.223665 -0.345039 -0.173506" rpy="0 0 0"/>
     <geometry>
       <mesh filename="package://robot_description/meshes/wheel_front_left_1.stl" scale="0.001 0.001 0.001"/>
@@ -113,10 +113,10 @@
 <link name="lidar_1">
   <inertial>
-    <origin xyz="2.534804336429275e-07 -3.095004238833077e-07 0.02952388194216904" rpy="0 0 0"/>
+    <origin xyz="-2.5348043358741634e-07 3.095004238833077e-07 0.02952388194216904" rpy="0 0 0"/>
     <mass value="100.3275293008071234"/>
-    <inertia ixx="0.001597" iyy="0.001597" izz="0.001837" ixy="-0.0" iyz="0.0" ixz="0.0"/>
+    <inertia ixx="0.001597" iyy="0.001597" izz="0.001837" ixy="-0.0" iyz="0.0" ixz="-0.0"/>
   </inertial>
   <visual>
-    <origin xyz="-0.308284 0.005039 -0.800004" rpy="0 0 0"/>
+    <origin xyz="0.308284 -0.005039 -0.800004" rpy="0 0 0"/>
     <geometry>
       <mesh filename="package://robot_description/meshes/lidar_1.stl" scale="0.001 0.001 0.001"/>
@@ -125,5 +125,5 @@
   </visual>
   <collision>
-    <origin xyz="-0.308284 0.005039 -0.800004" rpy="0 0 0"/>
+    <origin xyz="0.308284 -0.005039 -0.800004" rpy="0 0 0"/>
     <geometry>
       <mesh filename="package://robot_description/meshes/lidar_1.stl" scale="0.001 0.001 0.001"/>
@@ -132,5 +132,5 @@
 </link>
 <joint name="joint_back_left" type="continuous">
-  <origin xyz="0.353612 -0.345039 0.173506" rpy="0 0 0"/>
+  <origin xyz="-0.353612 0.345039 0.173506" rpy="0 0 0"/>
   <parent link="base_link"/>
   <child link="wheel_back_left_1"/>
@@ -140,5 +140,5 @@
 </joint>
 <joint name="joint_back_right" type="continuous">
-  <origin xyz="0.353612 0.334961 0.173506" rpy="0 0 0"/>
+  <origin xyz="-0.353612 -0.334961 0.173506" rpy="0 0 0"/>
   <parent link="base_link"/>
   <child link="wheel_back_right_1"/>
@@ -148,5 +148,5 @@
 </joint>
 <joint name="joint_front_right" type="continuous">
-  <origin xyz="-0.223665 0.334961 0.173506" rpy="0 0 0"/>
+  <origin xyz="0.223665 -0.334961 0.173506" rpy="0 0 0"/>
   <parent link="base_link"/>
   <child link="wheel_front_right_1"/>
@@ -156,5 +156,5 @@
 </joint>
 <joint name="joint_front_left" type="continuous">
-  <origin xyz="-0.223665 -0.345039 0.173506" rpy="0 0 0"/>
+  <origin xyz="0.223665 0.345039 0.173506" rpy="0 0 0"/>
   <parent link="base_link"/>
   <child link="wheel_front_left_1"/>
@@ -164,5 +164,5 @@
 </joint>
 <joint name="joint_lidar" type="fixed">
-  <origin xyz="0.308284 -0.005039 0.800004" rpy="0 0 0"/>
+  <origin xyz="-0.308284 0.005039 0.800004" rpy="0 0 0"/>
   <parent link="base_link"/>
   <child link="lidar_1"/>
